File: Hardware/Electronics/kicad/kicad.kicad_pcb (KiCad board)
At the start: 2 copper layers, 43.5 x 51.9 mm, 19 parts, among them J1 Conn_01x03_Socket, J6 USB_C_Receptacle_USB2.0_16P, Q1 BSS138, SW1 SW_Push, SW2 SW_Push, SW3 SW_Push, U1 USBLC6-2P6, U3 ESP32-C3-MINI-1-N4, U5 TLV1117-33

Commit message: Start on new PCB
Parts:
- added BT3: MY-ZJ-110, easyeda2kicad:SMD_MY-ZJ-110, F.Cu at (64.0, 152.2)
- added BT4: MY-ZJ-110, easyeda2kicad:SMD_MY-ZJ-110, F.Cu at (64.0, 81.8)
- added R6: 100k, Resistor_SMD:R_0603_1608Metric, F.Cu at (187.3, 103.7)
- moved SW3 99.2 mm to (64.0, 158.1)
- moved J1 3.85 mm to (169.6, 105.4)
Connections:
- net GND renamed -BATT
- SW3 pad 2: POI SW -> Net-(R6-Pad1)
Routing:
- net -BATT: track 133.3 -> 0.00 mm, vias 76 -> 0
- net +3.3V: track 110.7 -> 0.00 mm
- net +5V: track 82.0 -> 0.00 mm
- net POI SW: track 28.7 -> 0.00 mm
- net RESET: track 16.8 -> 0.00 mm
- net LED Data: track 16.5 -> 0.00 mm
- net +5VP: track 10.1 -> 0.00 mm
- net Net-(J1-Pin_2): track 8.48 -> 0.00 mm
- net Net-(J6-D+-PadA6): track 6.86 -> 0.00 mm
- net Net-(J6-D--PadA7): track 6.82 -> 0.00 mm
- net Net-(J6-CC1): track 5.78 -> 0.00 mm
- net BOOT: track 4.81 -> 0.00 mm
- net Net-(D1-A): track 4.12 -> 0.00 mm
- net USB_D+: track 3.54 -> 0.00 mm
- net USB_D-: track 3.42 -> 0.00 mm
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- removed copper zone on B.Cu, net -BATT
- removed copper zone on F.Cu, net -BATT
Other:
- board size 43.5 x 51.9 mm -> 28 x 130 mm

Commit message: Hardware Updates
Parts:
- added C2: 4.7n, Capacitor_SMD:C_0805_2012Metric, F.Cu at (75.8, 39.0)
- added C3: 4.7n, Capacitor_SMD:C_0805_2012Metric, F.Cu at (75.8, 45.8)
- added C4: 1u, Capacitor_SMD:C_0805_2012Metric, F.Cu at (57.2, 57.2)
- added C5: 1u, Capacitor_SMD:C_0805_2012Metric, F.Cu at (53.5, 61.5)
- added C8: 1u, Capacitor_SMD:C_0805_2012Metric, F.Cu at (53.5, 63.8)
- added C9: 22u, Capacitor_SMD:C_0805_2012Metric, F.Cu at (69.2, 62.0)
- added D2: LED, LED_SMD:LED_0603_1608Metric, F.Cu at (74.0, 47.8)
- added H1: MountingHole, MountingHole:MountingHole_3.2mm_M3_Pad, F.Cu at (53.5, 33.5)
- added H2: MountingHole, MountingHole:MountingHole_3.2mm_M3_Pad, F.Cu at (74.2, 33.5)
- added H3: MountingHole, MountingHole:MountingHole_3.2mm_M3_Pad, F.Cu at (53.5, 156.5)
- added H4: MountingHole, MountingHole:MountingHole_3.2mm_M3_Pad, F.Cu at (74.5, 156.5)
- added J2: Conn_01x03_Socket, Connector_JST:JST_PH_B3B-PH-K_1x03_P2.00mm_Vertical, F.Cu at (71.0, 74.7)
- added J3: Conn_01x03_Socket, Connector_JST:JST_PH_B3B-PH-K_1x03_P2.00mm_Vertical, F.Cu at (62.0, 74.7)
- added L1: XEL4030-102MEC, easyeda2kicad:IND-SMD_L4.0-W4.0-A, F.Cu at (74.0, 56.2)
- added R10: 220k, Resistor_SMD:R_0603_1608Metric, F.Cu at (61.0, 57.0)
- added R11: 100k, Resistor_SMD:R_0603_1608Metric, F.Cu at (74.8, 53.2)
- added R12: 100k, Resistor_SMD:R_0603_1608Metric, F.Cu at (74.2, 61.8)
- added R13: 732k, Resistor_SMD:R_0603_1608Metric, F.Cu at (74.2, 63.8)
- added R14: 10k, Resistor_SMD:R_0603_1608Metric, F.Cu at (74.8, 51.5)
- added R7: 2k, Resistor_SMD:R_0603_1608Metric, F.Cu at (72.5, 40.5)
- added R8: 1k, Resistor_SMD:R_0603_1608Metric, F.Cu at (74.0, 49.5)
- added R9: 220k, Resistor_SMD:R_0603_1608Metric, F.Cu at (59.2, 57.0)
- added U2: MCP73831-2-OT, Package_TO_SOT_SMD:SOT-23-5, F.Cu at (75.8, 42.5)
- added U4: XC6210B332MR, Package_TO_SOT_SMD:SOT-23-5, F.Cu at (54.0, 57.2)
- U5: value TLV1117-33 -> TPS61023DRLR; footprint Package_TO_SOT_SMD:SOT-223-3_TabPin2 -> easyeda2kicad:SOT-563_L1.6-W1.2-P0.50-LS1.6-BR
- moved R6 133.0 mm to (62.8, 57.0), turned to -90 degrees
- moved J1 120.5 mm to (53.0, 74.7)
- moved R4 110.0 mm to (66.0, 62.0), turned to -90 degrees
- moved Q1 109.3 mm to (64.0, 61.8)
- moved R1 105.5 mm to (60.8, 38.8)
- moved R3 104.9 mm to (69.0, 54.5), turned to 0 degrees
- moved SW1 104.2 mm to (69.2, 48.5), turned to -90 degrees
- moved SW2 103.6 mm to (69.2, 43.2), turned to -90 degrees
- moved C1 102.9 mm to (69.2, 52.5), turned to 180 degrees
- moved U3 99.7 mm to (58.7, 48.3)
- moved U1 98.7 mm to (64.5, 39.5)
- moved J6 98.4 mm to (64.0, 32.5)
- moved F1 98.3 mm to (68.2, 39.0)
- moved R2 98.2 mm to (60.8, 40.5)
- moved R5 95.8 mm to (64.5, 57.0), turned to 90 degrees
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Connections:
- net +5VP renamed Net-(F1-Pad1)
- C6 pad 2: +5V -> +BATT
- C7 pad 2: +3.3V -> +5V
- F1 pad 2: +5V -> +5VD
- J1 pad 1: +5V -> -BATT
- J1 pad 3: -BATT -> +5V
- R5 pad 2: +3.3V -> ESP LED
- R6 pad 1: Net-(R6-Pad1) -> POI SW
- R6 pad 2: POI SW -> +3.3V
- SW3 pad 2: Net-(R6-Pad1) -> POI SW
- U1 pad 5: +5V -> +5VD
- U3 pad 13: -BATT -> ESP LED
- U5 pad 1: -BATT -> Net-(U5-FB)
- U5 pad 2: +3.3V -> REG_SIGNAL
- U5 pad 3: +5V -> +BATT
Routing:
- net -BATT: track 0.00 -> 220.3 mm, vias 0 -> 72
- net POI SW: track 0.00 -> 125.5 mm, vias 0 -> 2
- net +BATT: track 0.00 -> 111.5 mm
- net +5V: track 0.00 -> 50.5 mm
- net Net-(J1-Pin_2): track 0.00 -> 37.5 mm
- net REG_SIGNAL: track 0.00 -> 29.4 mm, vias 0 -> 2
- net LED Data: track 0.00 -> 27.4 mm
- net +5VD: track 0.00 -> 26.0 mm
- net +3.3V: track 0.00 -> 23.3 mm
- net ESP LED: track 0.00 -> 17.6 mm
- net Net-(J6-CC1): track 0.00 -> 13.4 mm
- net Net-(F1-Pad1): track 0.00 -> 12.5 mm, vias 0 -> 2
- net RESET: track 0.00 -> 11.3 mm
- net Net-(J6-D--PadA7): track 0.00 -> 5.31 mm
- net Net-(U5-SW): track 0.00 -> 5.05 mm
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- added copper zone on B.Cu, net -BATT
- added copper zone on F.Cu, net -BATT
Other:
- board text added: "+5V"
- board text added: "BOOT"
- board text added: "GND"
- board text added: "LED"
- board text added: "OPEN PIXEL POI v2.2.0"
- board text added: "RESET"
- board text removed: "I designed this :)"
