File: Hardware/Electronics/kicad/kicad.kicad_sch (KiCad schematic)
At the start: 19 parts, among them J1 Conn_01x03_Socket, J6 USB_C_Receptacle_USB2.0_16P, Q1 BSS138, SW1 SW_Push, SW2 SW_Push, SW3 SW_Push, U1 USBLC6-2P6, U3 ESP32-C3-MINI-1-N4, U5 TLV1117-33

Commit message: Start on new PCB
Parts:
- added BT3, BT4: MY-ZJ-110, easyeda2kicad:SMD_MY-ZJ-110, symbol easyeda2kicad:MY-ZJ-110
- added R6: 100k, Resistor_SMD:R_0603_1608Metric, symbol Device:R_Small
Connections:
- net POI SW: now also R6.2; no longer SW3.2
- net GND renamed -BATT
- net -BATT: now also BT3.1
- new net: R6.1, SW3.2
- new net +BATT: BT4.1
Other:
- note added: "Battery Connectors"
- moved on the sheet: SW3
Changed lines of the file:
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@@
   (junction (at 57.15 34.29) (diameter 0) (color 0 0 0 0)
+  )
+  (junction (at 78.74 151.13) (diameter 0) (color 0 0 0 0)
   )
   (junction (at 20.32 67.31) (diameter 0) (color 0 0 0 0)
@@
     (stroke (width 0) (type default))
   )
+  (wire (pts (xy 72.39 151.13) (xy 78.74 151.13))
+    (stroke (width 0) (type default))
+  )
   (wire (pts (xy 199.39 52.07) (xy 203.2 52.07))
     (stroke (width 0) (type default))
@@
     (stroke (width 0) (type default))
   )
-  (wire (pts (xy 33.02 162.56) (xy 30.48 162.56))
-    (stroke (width 0) (type default))
-  )
   (wire (pts (xy 147.32 39.37) (xy 158.75 39.37))
     (stroke (width 0) (type default))
@@
     (stroke (width 0) (type default))
   )
+  (wire (pts (xy 52.07 153.67) (xy 53.34 153.67))
+    (stroke (width 0) (type default))
+  )
   (wire (pts (xy 203.2 87.63) (xy 203.2 85.09))
     (stroke (width 0) (type default))
@@
     (stroke (width 0) (type default))
   )
-  (wire (pts (xy 17.78 162.56) (xy 20.32 162.56))
-    (stroke (width 0) (type default))
-  )
   (wire (pts (xy 199.39 46.99) (xy 203.2 46.99))
     (stroke (width 0) (type default))
@@
     (stroke (width 0) (type default))
   )
+  (wire (pts (xy 78.74 151.13) (xy 80.01 151.13))
+    (stroke (width 0) (type default))
+  )
   (wire (pts (xy 199.39 41.91) (xy 203.2 41.91))
     (stroke (width 0) (type default))
@@
     (stroke (width 0) (type default))
   )
+  (rectangle (start 45.72 147.32) (end 100.33 157.48)
+    (stroke (width 0) (type default))
+    (fill (type none))
+  )
   (rectangle (start 45.72 118.11) (end 100.33 143.51)
     (stroke (width 0) (type default))
@@
     (stroke (width 0) (type default))
     (fill (type none))
+  )
+  (text "Battery Connectors" (at 46.99 147.32 0)
+    (effects (font (size 1.27 1.27)) (justify left bottom))
   )
   (text "LED Connector" (at 46.99 118.11 0)
@@
     )
   )
+  (symbol (lib_id "power:+BATT") (at 52.07 153.67 0) (unit 1)
+    (in_bom yes) (on_board yes) (dnp no) (fields_autoplaced)
+    (property "Reference" "#PWR015" (at 52.07 157.48 0)
+      (effects (font (size 1.27 1.27)) hide)
+    )
+    (property "Value" "+BATT" (at 52.07 148.59 0)
+      (effects (font (size 1.27 1.27)))
+    )
+    (property "Footprint" "" (at 52.07 153.67 0)
+      (effects (font (size 1.27 1.27)) hide)
+    )
+    (property "Datasheet" "" (at 52.07 153.67 0)
+      (effects (font (size 1.27 1.27)) hide)
+    )
+    (pin "1")
+    (instances
+      (project "kicad"
+        (path "/55a1363e-3506-4b1f-a7a5-0f5495c7c793"
+          (reference "#PWR015") (unit 1)
+        )
+      )
+    )
+  )
   (symbol (lib_id "power:GND") (at 17.78 162.56 0) (unit 1)
     (in_bom yes) (on_board yes) (dnp no) (fields_autoplaced)
@@
     )
   )
+  (symbol (lib_id "power:-BATT") (at 78.74 151.13 180) (unit 1)
+    (in_bom yes) (on_board yes) (dnp no)
+    (property "Reference" "#PWR023" (at 78.74 147.32 0)
+      (effects (font (size 1.27 1.27)) hide)
+    )
+    (property "Value" "-BATT" (at 76.2 156.21 0)
+      (effects (font (size 1.27 1.27)) (justify right))
+    )
+    (property "Footprint" "" (at 78.74 151.13 0)
+      (effects (font (size 1.27 1.27)) hide)
+    )
+    (property "Datasheet" "" (at 78.74 151.13 0)
+      (effects (font (size 1.27 1.27)) hide)
+    )
+    (pin "1")
+    (instances
+      (project "kicad"
+        (path "/55a1363e-3506-4b1f-a7a5-0f5495c7c793"
+          (reference "#PWR023") (unit 1)
+        )
+      )
+    )
+  )
   (symbol (lib_id "Switch:SW_Push") (at 25.4 149.86 0) (unit 1)
     (in_bom yes) (on_board yes) (dnp no) (fields_autoplaced)
@@
     )
   )
+  (symbol (lib_id "Device:R_Small") (at 30.48 162.56 90) (unit 1)
+    (in_bom yes) (on_board yes) (dnp no) (fields_autoplaced)
+    (property "Reference" "R6" (at 30.48 157.48 90)
+      (effects (font (size 1.27 1.27)))
+    )
+    (property "Value" "100k" (at 30.48 160.02 90)
+      (effects (font (size 1.27 1.27)))
+    )
+    (property "Footprint" "Resistor_SMD:R_0603_1608Metric" (at 30.48 162.56 0)
+      (effects (font (size 1.27 1.27)) hide)
+    )
+    (property "Datasheet" "~" (at 30.48 162.56 0)
+      (effects (font (size 1.27 1.27)) hide)
+    )
+    (property "LCSC" "C14675" (at 30.48 162.56 0)
+      (effects (font (size 1.27 1.27)) hide)
+    )
+    (pin "1")
+    (pin "2")
+    (instances
+      (project "kicad"
+        (path "/55a1363e-3506-4b1f-a7a5-0f5495c7c793"
+          (reference "R6") (unit 1)
+        )
+      )
+    )
+  )
   (symbol (lib_id "power:GND") (at 154.94 113.03 0) (unit 1)
     (in_bom yes) (on_board yes) (dnp no) (fields_autoplaced)
@@
     )
   )
+  (symbol (lib_id "easyeda2kicad:MY-ZJ-110") (at 83.82 151.13 0) (unit 1)
+    (in_bom yes) (on_board yes) (dnp no) (fields_autoplaced)
+    (property "Reference" "BT3" (at 88.9 149.86 0)
+      (effects (font (size 1.27 1.27)) (justify left))
+    )
+    (property "Value" "MY-ZJ-110" (at 88.9 152.4 0)
+      (effects (font (size 1.27 1.27)) (justify left) hide)
+    )
+    (property "Footprint" "easyeda2kicad:SMD_MY-ZJ-110" (at 83.82 158.75 0)
+      (effects (font (size 1.27 1.27)) hide)
+    )
+    (property "Datasheet" "" (at 83.82 151.13 0)
+      (effects (font (size 1.27 1.27)) hide)
+    )
+    (property "LCSC Part" "C964859" (at 83.82 161.29 0)
+      (effects (font (size 1.27 1.27)) hide)
+    )
+    (pin "1")
+    (instances
+      (project "kicad"
+        (path "/55a1363e-3506-4b1f-a7a5-0f5495c7c793"
+          (reference "BT3") (unit 1)
+        )
+      )
+    )
+  )
   (symbol (lib_id "power:GND") (at 59.69 34.29 0) (unit 1)
     (in_bom yes) (on_board yes) (dnp no) (fields_autoplaced)
@@
     )
   )
-  (symbol (lib_id "Switch:SW_Push") (at 25.4 162.56 0) (unit 1)
-    (in_bom yes) (on_board yes) (dnp no) (fields_autoplaced)
-    (property "Reference" "SW3" (at 25.4 154.94 0)
-      (effects (font (size 1.27 1.27)))
-    )
-    (property "Value" "SW_Push" (at 25.4 157.48 0)
-      (effects (font (size 1.27 1.27)))
-    )
-    (property "Footprint" "Button_Switch_SMD:Panasonic_EVQPUL_EVQPUC" (at 25.4 157.48 0)
-      (effects (font (size 1.27 1.27)) hide)
-    )
-    (property "Datasheet" "~" (at 25.4 157.48 0)
-      (effects (font (size 1.27 1.27)) hide)
-    )
-    (property "LCSC" "C79174" (at 25.4 162.56 0)
+  (symbol (lib_id "Switch:SW_Push") (at 22.86 162.56 0) (unit 1)
+    (in_bom yes) (on_board yes) (dnp no) (fields_autoplaced)
+    (property "Reference" "SW3" (at 22.86 154.94 0)
+      (effects (font (size 1.27 1.27)))
+    )
+    (property "Value" "SW_Push" (at 22.86 157.48 0)
+      (effects (font (size 1.27 1.27)))
+    )
+    (property "Footprint" "Button_Switch_SMD:Panasonic_EVQPUL_EVQPUC" (at 22.86 157.48 0)
+      (effects (font (size 1.27 1.27)) hide)
+    )
+    (property "Datasheet" "~" (at 22.86 157.48 0)
+      (effects (font (size 1.27 1.27)) hide)
+    )
+    (property "LCSC" "C79174" (at 22.86 162.56 0)
       (effects (font (size 1.27 1.27)) hide)
     )
@@
     )
   )
+  (symbol (lib_id "power:GND") (at 72.39 151.13 0) (unit 1)
+    (in_bom yes) (on_board yes) (dnp no) (fields_autoplaced)
+    (property "Reference" "#PWR024" (at 72.39 157.48 0)
+      (effects (font (size 1.27 1.27)) hide)
+    )
+    (property "Value" "GND" (at 72.39 156.21 0)
+      (effects (font (size 1.27 1.27)))
+    )
+    (property "Footprint" "" (at 72.39 151.13 0)
+      (effects (font (size 1.27 1.27)) hide)
+    )
+    (property "Datasheet" "" (at 72.39 151.13 0)
+      (effects (font (size 1.27 1.27)) hide)
+    )
+    (pin "1")
+    (instances
+      (project "kicad"
+        (path "/55a1363e-3506-4b1f-a7a5-0f5495c7c793"
+          (reference "#PWR024") (unit 1)
+        )
+      )
+    )
+  )
   (symbol (lib_id "power:GND") (at 20.32 100.33 0) (unit 1)
     (in_bom yes) (on_board yes) (dnp no) (fields_autoplaced)
@@
         )
       )
+    )
+  )
+  (symbol (lib_id "easyeda2kicad:MY-ZJ-110") (at 57.15 153.67 0) (unit 1)
+    (in_bom yes) (on_board yes) (dnp no) (fields_autoplaced)
+    (property "Reference" "BT4" (at 62.23 152.4 0)
+      (effects (font (size 1.27 1.27)) (justify left))
+    )
+    (property "Value" "MY-ZJ-110" (at 62.23 154.94 0)
+      (effects (font (size 1.27 1.27)) (justify left) hide)
+    )
+    (property "Footprint" "easyeda2kicad:SMD_MY-ZJ-110" (at 57.15 161.29 0)
+      (effects (font (size 1.27 1.27)) hide)
+    )
+    (property "Datasheet" "" (at 57.15 153.67 0)
+      (effects (font (size 1.27 1.27)) hide)
+    )
+    (property "LCSC Part" "C964859" (at 57.15 163.83 0)
+      (effects (font (size 1.27 1.27)) hide)
+    )
+    (pin "1")
+    (instances
+      (project "kicad"
+        (path "/55a1363e-3506-4b1f-a7a5-0f5495c7c793"
+          (reference "BT4") (unit 1)
+        )
+      )

Commit message: Hardware Updates
Parts:
- removed U5: TLV1117-33, Package_TO_SOT_SMD:SOT-223-3_TabPin2, symbol Regulator_Linear:TLV1117-33
- added C2, C3: 4.7n, Capacitor_SMD:C_0805_2012Metric, symbol Device:C_Small
- added C4, C5, C8: 1u, Capacitor_SMD:C_0805_2012Metric, symbol Device:C_Small
- added C9: 22u, Capacitor_SMD:C_0805_2012Metric, symbol Device:C_Small
- added D2: LED, LED_SMD:LED_0603_1608Metric, symbol Device:LED
- added H1, H2, H3, H4: MountingHole, MountingHole:MountingHole_3.2mm_M3_Pad, symbol Mechanical:MountingHole_Pad
- added J2, J3: Conn_01x03_Socket, Connector_JST:JST_PH_B3B-PH-K_1x03_P2.00mm_Vertical, symbol Connector:Conn_01x03_Socket
- added L1: XEL4030-102MEC, easyeda2kicad:IND-SMD_L4.0-W4.0-A, symbol easyeda2kicad:XEL4030-102MEC
- added R10, R9: 220k, Resistor_SMD:R_0603_1608Metric, symbol Device:R_Small
- added R11, R12: 100k, Resistor_SMD:R_0603_1608Metric, symbol Device:R_Small
- added R13: 732k, Resistor_SMD:R_0603_1608Metric, symbol Device:R_Small
- added R14: 10k, Resistor_SMD:R_0603_1608Metric, symbol Device:R_Small
- added R7: 2k, Resistor_SMD:R_0603_1608Metric, symbol Device:R_Small
- added R8: 1k, Resistor_SMD:R_0603_1608Metric, symbol Device:R_Small
- added U2: MCP73831-2-OT, Package_TO_SOT_SMD:SOT-23-5, symbol Battery_Management:MCP73831-2-OT
- added U4: XC6210B332MR, Package_TO_SOT_SMD:SOT-23-5, symbol Regulator_Linear:XC6210B332MR
- added U5: TPS61023DRLR, easyeda2kicad:SOT-563_L1.6-W1.2-P0.50-LS1.6-BR, symbol easyeda2kicad:TPS61023DRLR
- BT3, BT4: LCSC (none) -> C964859
- C6, C7: LCSC C86816 -> C45783
Connections:
- net +3.3V: now also R6.2, C4.2, U4.5 (VOUT); no longer C7.2, R5.2
- net +5V: now also C7.2, J1.3 (Pin_3), C9.2, J2.3 (Pin_3), J3.3 (Pin_3), R13.2, U5.6 (VOUT); no longer C6.2, F1.2, J1.1 (Pin_1), U1.5 (VBUS)
- net +BATT: now also C6.2, C3.2, C5.2, C8.2, L1.1, R11.1, R9.2, U2.3 (V_{BAT}), U4.1 (VIN), U4.3 (CE), U5.3 (VIN)
- net -BATT: now also J1.1 (Pin_1), C2.1, C3.1, C4.1, C5.1, C8.1, C9.1, H1.1, H2.1, H3.1, H4.1, J2.1 (Pin_1), J3.1 (Pin_1), R10.1, R12.1, R14.2, R7.2, U2.2 (V_{SS}), U4.2 (GND), U5.4 (GND); no longer J1.3 (Pin_3), U3.13 (IO1)
- net POI SW: now also R6.1, SW3.2; no longer R6.2
- net REG_SIGNAL: now also R11.2, R14.1, U5.2 (EN)
- net VBATT_SENSE: now also R10.2, R9.1
- net at J1.2 (Pin_2), Q1.3 (D), R4.1: now also J2.2 (Pin_2), J3.2 (Pin_2)
- net +5VP: no longer names the net of F1.1, J6.A4 (VBUS), J6.A9 (VBUS), J6.B4 (VBUS), J6.B9 (VBUS)
- new net: D2.1 (K), U2.1 (STAT)
- new net: D2.2 (A), R8.1
- new net: L1.2, U5.5 (SW)
- new net: R7.1, U2.5 (PROG)
- new net: R12.2, R13.1, U5.1 (FB)
- new net +5VD: C2.2, F1.2, R8.2, U1.5 (VBUS), U2.4 (V_{DD})
- new net ESP LED: R5.2, U3.13 (IO1)
Other:
- note added: "5v Regulator"
- note added: "Batt Voltage Divider"
- note added: "Battery Charger"
- note added: "ESP Power LED"
- note added: "Mounting Holes"
- note removed: "3.3v Power LED"
- moved on the sheet: BT3, BT4, C1, D1, J1, Q1, R3, R4, R5, R6, SW1, SW2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
