File: Hardware/Electronics/kicad/kicad.kicad_sch (KiCad schematic)
At the start: 47 parts, among them J1 Conn_01x03_Socket, J2 Conn_01x03_Socket, J3 Conn_01x03_Socket, J6 USB_C_Receptacle_USB2.0_16P, SW1 SW_Push, SW2 SW_Push, SW3 SW_Push, U1 USBLC6-2P6, U2 MCP73831-2-OT, U3 ESP32-C3-MINI-1-N4, U4 XC6210B332MR, U5 TPS61023DRLR, U6 SN74LV1T34DBV

Commit message: PCB Tweaks
Parts:
- SW3: LCSC C79174 -> C397351
Changed lines of the file:
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@@
       (effects (font (size 1.27 1.27)) hide)
     )
-    (property "Datasheet" "" (at 144.78 113.03 0)
+    (property "Datasheet" "Backup part # C19188671" (at 144.78 113.03 0)
       (effects (font (size 1.27 1.27)) hide)
     )
@@
       (effects (font (size 1.27 1.27)) hide)
     )
-    (property "LCSC" "C79174" (at 21.59 158.75 0)
-      (effects (font (size 1.27 1.27)) hide)
-    )
+    (property "LCSC" "C397351" (at 21.59 158.75 0)
+      (effects (font (size 1.27 1.27)) hide)
+    )

Commit message: Add KiCad MCP configuration and new script for editing schematic text
- Introduced a new MCP configuration file for KiCad.
- Added a Python script to automate the editing of schematic text, including functionality for managing component instances and labels.
- Updated the platformio.ini to streamline the default environment settings.
- Adjusted firmware BLE handling for pattern saving and button state management.
- Modified LED handling to support multiple strips and improved brightness control.
- Updated KiCad PCB files and removed obsolete autosave files.
Parts:
- removed BT3, BT4: MY-ZJ-110, easyeda2kicad:SMD_MY-ZJ-110, symbol easyeda2kicad:MY-ZJ-110
- removed H1, H2, H3, H4: MountingHole, MountingHole:MountingHole_3.2mm_M3_Pad, symbol Mechanical:MountingHole_Pad
- removed J1, J2, J3: Conn_01x03_Socket, Connector_JST:JST_PH_B3B-PH-K_1x03_P2.00mm_Vertical, symbol Connector:Conn_01x03_Socket
- removed SW3: SW_Push, Button_Switch_SMD:Panasonic_EVQPUL_EVQPUC, symbol Switch:SW_Push
- added J7: Batt+Btn, custom_footprints:Power_Button_SolderPads_1x03, symbol Connector:Conn_01x03_Socket
- added J8, J9: LED, custom_footprints:LED_Strip_SolderPads_1x04, symbol Connector:Conn_01x04_Socket
- added U7: SN74LV1T34DBV, Package_TO_SOT_SMD:SOT-23-5, symbol Logic_LevelTranslator:SN74LV1T34DBV
Connections:
- net +5V: now also J8.2 (Pin_2), J9.2 (Pin_2), U7.5 (VCC)
- net +BATT: now also J7.1 (Pin_1)
- net -BATT: now also J7.2 (Pin_2), J8.1 (Pin_1), J9.1 (Pin_1), U7.3 (GND)
- net POI SW: now also J7.3 (Pin_3)
- net LED1: now reaches U6.4 (Y)
- net LED1: now also J8.3 (Pin_3), J9.3 (Pin_3)
- new net LED Data 2: U7.2 (A)
- new net LED2: J8.4 (Pin_4), J9.4 (Pin_4), U7.4 (Y)
- no-connect marks 14 -> 15
