File: Hardware/Electronics/kicad/_autosave-kicad.kicad_sch (KiCad schematic)
At the start: 47 parts, among them J1 Conn_01x03_Socket, J2 Conn_01x03_Socket, J3 Conn_01x03_Socket, J6 USB_C_Receptacle_USB2.0_16P, SW1 SW_Push, SW2 SW_Push, SW3 SW_Push, U1 USBLC6-2P6, U2 MCP73831-2-OT, U3 ESP32-C3-MINI-1-N4, U4 XC6210B332MR, U5 TPS61023DRLR, U6 SN74LV1T34DBV

Commit message: Hardware 2.2.1
Parts:
- C2, C3: LCSC C1744 -> C123621
Changed lines of the file:
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@@
       (effects (font (size 1.27 1.27)) hide)
     )
-    (property "LCSC" "C1744" (at 87.63 170.18 0)
+    (property "LCSC" "C123621" (at 87.63 170.18 0)
       (effects (font (size 1.27 1.27)) hide)
     )
@@
       (effects (font (size 1.27 1.27)) hide)
     )
-    (property "LCSC" "C1744" (at 46.99 166.37 0)
-      (effects (font (size 1.27 1.27)) hide)
-    )
+    (property "LCSC" "C123621" (at 46.99 166.37 0)
+      (effects (font (size 1.27 1.27)) hide)
+    )
